Commit message: Fetch robot doesnt explode anymore.
Had to set damping to zero which... doesn't make sense. Damping I thought was supposed to determine how fast a rotation slows down, but right now the rotation only slows down if damping is 0

Removed the collision for the target cube. Will be manually checking target collision

File: pybulletgym/envs/assets/things/cubes/cube_target_no_collision.urdf (robot description, URDF)
Before this commit: robot cube_target.urdf, 1 links, 0 joints
Links:
- link baseLink: geometry visual box size=.1 .1 .1
