Commit message: Started knife / cube cut behavior

File: pybulletgym/envs/assets/things/cubes/cube_target_basic.urdf (robot description, URDF)
Before this commit: robot cube_concave.urdf, 1 links, 0 joints
Links:
- removed link cube_concave_base_link
- added link baseLink, mass 0; collision box size=.1 .1 .1; visual box size=.1 .1 .1

File: pybulletgym/envs/assets/things/knives/knife.urdf (robot description, URDF)
Before this commit: robot knife.urdf, 2 links, 1 joints
Joints:
- removed joint head_camera_depth_joint
- added joint handle_to_blade_joint: type fixed, parent handle, child blade, origin xyz=0 0 0 rpy=0 0 0
