Commit message: Made Knife Bigger... Added reward augment decorator Added velocity augment for set_position (prevent jerking motion)

File: pybulletgym/envs/assets/things/knives/knife.urdf (robot description, URDF)
Before this commit: robot knife.urdf, 2 links, 1 joints
Links:
- link blade: geometry collision mesh filename=knife_blade.obj scale=.02 .02 .02; visual mesh filename=knife_blade.obj scale=.02 .02 .02
- link handle: geometry collision mesh filename=knife_handle.obj scale=.021 .021 .021; visual mesh filename=knife_handle.obj scale=.02 .02 .02
