Commit message: URDF parsing is working, and running. I want the textures to load with the DAE. I confirmed that they load, but the images don't. Going to test obj conversion and see if the textures show up then

File: pybulletgym/envs/assets/robots/fetch/fetch_description/robots/fetch.urdf (robot description, URDF)
Before this commit: robot fetch, 26 links, 25 joints
Links:
- link head_camera_depth_frame: mass None -> 0
- link head_camera_depth_optical_frame: mass None -> 0
- link head_camera_link: mass None -> 0
- link head_camera_rgb_frame: mass None -> 0
- link head_camera_rgb_optical_frame: mass None -> 0

Commit message: Went into blender, converted all the dae's into obj's. I kept the dae, however the urdf is now targeting the obj extensions instead.
As to why the robot is a blue tint I will need to find out..

File: pybulletgym/envs/assets/robots/fetch/fetch_description/robots/fetch.urdf (robot description, URDF)
Before this commit: robot fetch, 26 links, 25 joints
Links:
- link base_link: geometry collision mesh filename=package://fetch_description/meshes/base_link_collision.STL; visual mesh filename=package://fetch_description/meshes/base_link.obj
- link elbow_flex_link: geometry collision mesh filename=package://fetch_description/meshes/elbow_flex_link_collisio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; visual mesh filename=package://fetch_description/meshes/elbow_flex_link.obj
- link forearm_roll_link: geometry collision mesh filename=package://fetch_description/meshes/forearm_roll_link_collis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; visual mesh filename=package://fetch_description/meshes/forearm_roll_link.obj
- link gripper_link: geometry collision mesh filename=package://fetch_description/meshes/gripper_link.STL; visual mesh filename=package://fetch_description/meshes/gripper_link.obj
- link head_pan_link: geometry collision mesh filename=package://fetch_description/meshes/head_pan_link_collision.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; visual mesh filename=package://fetch_description/meshes/head_pan_link.obj
- link head_tilt_link: geometry collision mesh filename=package://fetch_description/meshes/head_tilt_link_collision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; visual mesh filename=package://fetch_description/meshes/head_tilt_link.obj
- link shoulder_lift_link: geometry collision mesh filename=package://fetch_description/meshes/shoulder_lift_link_colli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; visual mesh filename=package://fetch_description/meshes/shoulder_lift_link.obj
- link shoulder_pan_link: geometry collision mesh filename=package://fetch_description/meshes/shoulder_pan_link_collis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; visual mesh filename=package://fetch_description/meshes/shoulder_pan_link.obj
- link torso_fixed_link: geometry collision mesh filename=package://fetch_description/meshes/torso_fixed_link.STL; visual mesh filename=package://fetch_description/meshes/torso_fixed_link.obj
- link torso_lift_link: geometry collision mesh filename=package://fetch_description/meshes/torso_lift_link_collisio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; visual mesh filename=package://fetch_description/meshes/torso_lift_link.obj
- link upperarm_roll_link: geometry collision mesh filename=package://fetch_description/meshes/upperarm_roll_link_colli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; visual mesh filename=package://fetch_description/meshes/upperarm_roll_link.obj
- link wrist_flex_link: geometry collision mesh filename=package://fetch_description/meshes/wrist_flex_link_collisio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; visual mesh filename=package://fetch_description/meshes/wrist_flex_link.obj
- link wrist_roll_link: geometry collision mesh filename=package://fetch_description/meshes/wrist_roll_link_collisio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; visual mesh filename=package://fetch_description/meshes/wrist_roll_link.obj

Commit message: RL works now
Need to change it to floats. The NN needs to be able adjust the power to the joints. They are either at 100% or 0% lol

File: pybulletgym/envs/assets/robots/fetch/fetch_description/robots/fetch.urdf (robot description, URDF)
Before this commit: robot fetch, 26 links, 25 joints
Joints:
- joint elbow_flex_joint: origin xyz=0.133 0 0 rpy=0 0 0 -> xyz=0.133 0 0 rpy=0 -1.5 0
- joint forearm_roll_joint: origin xyz=0.197 0 0 rpy=0 0 0 -> xyz=0.197 0 0 rpy=1.5 0 0
- joint shoulder_lift_joint: origin xyz=0.117 0 0.0599999999999999 rpy=0 0 0 -> xyz=0.117 0 0.0599999999999999 rpy=0 1.5 0
- joint shoulder_pan_joint: origin xyz=0.119525 0 0.34858 rpy=0 0 0 -> xyz=0.119525 0 0.34858 rpy=0 0 -1.5
- joint upperarm_roll_joint: origin xyz=0.219 0 0 rpy=0 0 0 -> xyz=0.219 0 0 rpy=3 0 0

Commit message: Saving fetch.urdf edit

File: pybulletgym/envs/assets/robots/fetch/fetch_description/robots/fetch.urdf (robot description, URDF)
Before this commit: robot fetch, 26 links, 25 joints
Links:
- removed link elbow_flex_link
- removed link estop_link
- removed link forearm_roll_link
- removed link gripper_link
- removed link head_camera_depth_frame
- removed link head_camera_depth_optical_frame
- removed link head_camera_link
- removed link head_camera_rgb_frame
- removed link head_camera_rgb_optical_frame
- removed link l_gripper_finger_link
- removed link laser_link
- removed link r_gripper_finger_link
- removed link shoulder_lift_link
- removed link shoulder_pan_link
- removed link upperarm_roll_link
- removed link wrist_flex_link
- removed link wrist_roll_link
- link torso_lift_link: geometry collision mesh filename=package://fetch_description/meshes/torso_lift_link_collisio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 scale=0.7 1 1; visual mesh filename=package://fetch_description/meshes/torso_lift_link.obj
Joints:
- removed joint elbow_flex_joint
- removed joint estop_joint
- removed joint forearm_roll_joint
- removed joint gripper_axis
- removed joint head_camera_depth_joint
- removed joint head_camera_depth_optical_joint
- removed joint head_camera_joint
- removed joint head_camera_rgb_joint
- removed joint head_camera_rgb_optical_joint
- removed joint l_gripper_finger_joint
- removed joint laser_joint
- removed joint r_gripper_finger_joint
- removed joint shoulder_lift_joint
- removed joint shoulder_pan_joint
- removed joint upperarm_roll_joint
- removed joint wrist_flex_joint
- removed joint wrist_roll_joint
- joint l_wheel_joint: origin xyz=0.0012914 0.18738 0.055325 rpy=-6.123E-17 0 0 -> xyz=0.0012914 0.18738 0.060325 rpy=-6.123E-17 0 0
- joint r_wheel_joint: origin xyz=0.0012914 -0.18738 0.055325 rpy=-6.123E-17 0 0 -> xyz=0.0012914 -0.18738 0.060325 rpy=-6.123E-17 0 0

Commit message: Fetch URDF works now. Does not explode.
Needed to fix collision boxes. I think that the bullet3 margin is different from a Gazebo margin.

File: pybulletgym/envs/assets/robots/fetch/fetch_description/robots/fetch.urdf (robot description, URDF)
Before this commit: robot fetch, 9 links, 8 joints
Links:
- added link elbow_flex_link, mass 2.1299; collision mesh filename=package://fetch_description/meshes/elbow_flex_link_collisio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 scale=1 1 1; visual mesh filename=package://fetch_description/meshes/elbow_flex_link.obj
- added link estop_link, mass 0.00196130439134723; collision mesh filename=package://fetch_description/meshes/estop_link.STL; visual mesh filename=package://fetch_description/meshes/estop_link.STL
- added link forearm_roll_link, mass 1.6563; collision mesh filename=package://fetch_description/meshes/forearm_roll_link_collis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 scale=1 1 1; visual mesh filename=package://fetch_description/meshes/forearm_roll_link.obj
- added link gripper_link, mass 1.5175; collision mesh filename=package://fetch_description/meshes/gripper_link.STL; visual mesh filename=package://fetch_description/meshes/gripper_link.obj
- added link head_camera_depth_frame, mass 0
- added link head_camera_depth_optical_frame, mass 0
- added link head_camera_link, mass 0
- added link head_camera_rgb_frame, mass 0
- added link head_camera_rgb_optical_frame, mass 0
- added link l_gripper_finger_link, mass 0.0798; collision mesh filename=package://fetch_description/meshes/l_gripper_finger_link.STL; visual mesh filename=package://fetch_description/meshes/l_gripper_finger_link.STL
- added link laser_link, mass 0.00833634573995571; collision mesh filename=package://fetch_description/meshes/laser_link.STL; visual mesh filename=package://fetch_description/meshes/laser_link.STL
- added link r_gripper_finger_link, mass 0.0798; collision mesh filename=package://fetch_description/meshes/r_gripper_finger_link.STL; visual mesh filename=package://fetch_description/meshes/r_gripper_finger_link.STL
- added link shoulder_lift_link, mass 2.6615; collision mesh filename=package://fetch_description/meshes/shoulder_lift_link_colli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 scale=1 1 0.8; visual mesh filename=package://fetch_description/meshes/shoulder_lift_link.obj
- added link shoulder_pan_link, mass 2.5587; collision mesh filename=package://fetch_description/meshes/shoulder_pan_link_collis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; visual mesh filename=package://fetch_description/meshes/shoulder_pan_link.obj
- added link upperarm_roll_link, mass 2.3311; collision mesh filename=package://fetch_description/meshes/upperarm_roll_link_colli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 scale=1 1 0.8; visual mesh filename=package://fetch_description/meshes/upperarm_roll_link.obj
- added link wrist_flex_link, mass 1.725; collision mesh filename=package://fetch_description/meshes/wrist_flex_link_collisio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; visual mesh filename=package://fetch_description/meshes/wrist_flex_link.obj
- added link wrist_roll_link, mass 0.1354; collision mesh filename=package://fetch_description/meshes/wrist_roll_link_collisio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; visual mesh filename=package://fetch_description/meshes/wrist_roll_link.obj
- link bellows_link2: geometry visual mesh filename=package://fetch_description/meshes/bellows_link.STL
Joints:
- added joint elbow_flex_joint: type revolute, parent upperarm_roll_link, child elbow_flex_link, origin xyz=0.133 0 0 rpy=0 -1.8 0, axis 0 1 0, limit lower=-2.251 upper=2.251 effort=66.18 velocity=1.521
- added joint estop_joint: type fixed, parent base_link, child estop_link, origin xyz=-0.12465 0.23892 0.31127 rpy=1.5708 0 0, axis 0 0 0
- added joint forearm_roll_joint: type continuous, parent elbow_flex_link, child forearm_roll_link, origin xyz=0.197 0 0 rpy=0 0 0, axis 1 0 0, limit effort=29.35 velocity=1.571
- added joint gripper_axis: type fixed, parent wrist_roll_link, child gripper_link, origin xyz=0.16645 0 0 rpy=0 0 0, axis 0 1 0
- added joint head_camera_depth_joint: type fixed, parent head_camera_link, child head_camera_depth_frame, origin xyz=0 0.045 0 rpy=0 0 0
- added joint head_camera_depth_optical_joint: type fixed, parent head_camera_depth_frame, child head_camera_depth_optical_frame, origin xyz=0 0 0 rpy=-1.57079632679 0 -1.57079632679
- added joint head_camera_joint: type fixed, parent head_tilt_link, child head_camera_link, origin xyz=0.055 0 0.0225 rpy=0 0 0
- added joint head_camera_rgb_joint: type fixed, parent head_camera_link, child head_camera_rgb_frame, origin xyz=0 0.02 0 rpy=0 0 0
- added joint head_camera_rgb_optical_joint: type fixed, parent head_camera_rgb_frame, child head_camera_rgb_optical_frame, origin xyz=0 0 0 rpy=-1.57079632679 0 -1.57079632679
- added joint l_gripper_finger_joint: type prismatic, parent gripper_link, child l_gripper_finger_link, origin xyz=0 -0.015425 0 rpy=0 0 0, axis 0 -1 0, limit lower=0.0 upper=0.05 effort=60 velocity=0.05
- added joint laser_joint: type fixed, parent base_link, child laser_link, origin xyz=0.235 0 0.2878 rpy=3.14159265359 0 0, axis 0 0 0
- added joint r_gripper_finger_joint: type prismatic, parent gripper_link, child r_gripper_finger_link, origin xyz=0 0.015425 0 rpy=0 0 0, axis 0 1 0, limit lower=0.0 upper=0.05 effort=60 velocity=0.05
- added joint shoulder_lift_joint: type revolute, parent shoulder_pan_link, child shoulder_lift_link, origin xyz=0.117 0.0 0.0599999999999999 rpy=0 1.5 0, axis 0 1 0, limit lower=-1.221 upper=1.518 effort=131.76 velocity=1.454
- added joint shoulder_pan_joint: type revolute, parent torso_lift_link, child shoulder_pan_link, origin xyz=0.119525 0 0.34858 rpy=0 0 -1.5, axis 0 0 1, limit lower=-1.6056 upper=1.6056 effort=33.82 velocity=1.256
- added joint upperarm_roll_joint: type continuous, parent shoulder_lift_link, child upperarm_roll_link, origin xyz=0.219 0 0 rpy=3.3 0 0, axis 1 0 0, limit effort=76.94 velocity=1.571
- added joint wrist_flex_joint: type revolute, parent forearm_roll_link, child wrist_flex_link, origin xyz=0.1245 0 0 rpy=0 -1.5 0, axis 0 1 0, limit lower=-2.16 upper=2.16 effort=25.7 velocity=2.268
- added joint wrist_roll_joint: type continuous, parent wrist_flex_link, child wrist_roll_link, origin xyz=0.1385 0 0 rpy=0 0 0, axis 1 0 0, limit effort=7.36 velocity=2.268

Commit message: Removed set joints int he URDf. Was screwing up the joint limits

File: pybulletgym/envs/assets/robots/fetch/fetch_description/robots/fetch.urdf (robot description, URDF)
Before this commit: robot fetch, 26 links, 25 joints
Joints:
- joint elbow_flex_joint: origin xyz=0.133 0 0 rpy=0 -1.8 0 -> xyz=0.133 0 0 rpy=0 0 0
- joint shoulder_lift_joint: origin xyz=0.117 0.0 0.0599999999999999 rpy=0 1.5 0 -> xyz=0.117 0.0 0.0599999999999999 rpy=0 0 0
- joint shoulder_pan_joint: origin xyz=0.119525 0 0.34858 rpy=0 0 -1.5 -> xyz=0.119525 0 0.34858 rpy=0 0 0
- joint wrist_flex_joint: origin xyz=0.1245 0 0 rpy=0 -1.5 0 -> xyz=0.1245 0 0 rpy=0 0 0

Commit message: Updating develop_2 branch.
Added no-friction behavior.

Changed base envs to be more similar to openai implementation.

Changed default action input to position based

File: pybulletgym/envs/assets/robots/fetch/fetch_description/robots/fetch.urdf (robot description, URDF)
Before this commit: robot fetch, 26 links, 25 joints
Joints:
- joint upperarm_roll_joint: origin xyz=0.219 0 0 rpy=3.3 0 0 -> xyz=0.219 0 0 rpy=3.15 0 0

File: pybulletgym/envs/assets/things/cubes/cube_no_friction_projectile.urdf (robot description, URDF)
Before this commit: robot urdf_cube_target, 1 links, 0 joints
Links:
- link base_link: mass 10 -> 1
